File: mega shield/mega shield.sch (KiCad schematic (older format))
At the start: 30 parts, among them J1 Conn_01x08_Male, J10 Conn_01x04_Male, J11 Conn_01x04_Male, J12 Conn_01x04_Male, J13 Conn_01x03_Male, J14 Conn_01x03_Male, J15 Conn_01x03_Male, J16 Conn_01x03_Male, J17 POWER IN, J18 3.3V OUT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

Commit message: mega shield completed
Parts:
- removed J10, J8, J9: Conn_01x04_Male, Connector_JST:JST_EH_B4B-EH-A_1x04_P2.50mm_Vertical, symbol Connector:Conn_01x04_Male
- added J10: Conn_01x08_Male, Connector_JST:JST_EH_B8B-EH-A_1x08_P2.50mm_Vertical, symbol Connector:Conn_01x08_Male
- added J19: Conn_01x04_Male, Connector_JST:JST_EH_B4B-EH-A_1x04_P2.50mm_Vertical, symbol Connector:Conn_01x04_Male
- added J20: Conn_01x03_Male, Connector_JST:JST_EH_B3B-EH-A_1x03_P2.50mm_Vertical, symbol Connector:Conn_01x03_Male
- added J8: Conn_01x02_Male, Connector_JST:JST_EH_B2B-EH-A_1x02_P2.50mm_Vertical, symbol Connector:Conn_01x02_Male
- D1: footprint Diode_THT:D_A-405_P10.16mm_Horizontal -> Diode_THT:D_DO-27_P15.24mm_Horizontal
- SW1: footprint Resistor_THT:R_Axial_DIN0207_L6.3mm_D2.5mm_P7.62mm_Horizontal -> Button_Switch_THT:SW_PUSH_6mm_H5mm
Connections:
- net +3V3: now also J18.1 (Pin_1); no longer J18.2 (Pin_2)
- net +5V: now also J12.2 (Pin_2), R1.1, J10.1 (Pin_1), J19.2 (Pin_2), J20.2 (Pin_2); no longer J12.3 (Pin_3)
- net A0: now also J10.3 (Pin_3); no longer J13.1 (Pin_1)
- net A1: now also J10.4 (Pin_4); no longer J14.1 (Pin_1)
- net A10: now also J4.5 (Pin_5); no longer J4.7 (Pin_7)
- net A11: now also J4.6 (Pin_6); no longer J4.8 (Pin_8)
- net A12: now also J4.7 (Pin_7); no longer J5.1 (Pin_1)
- net A13: now also J4.8 (Pin_8); no longer J5.2 (Pin_2)
- net A14: now also J5.1 (Pin_1); no longer J5.3 (Pin_3)
- net A15: now also J5.2 (Pin_2); no longer J5.4 (Pin_4)
- net A2: now also J10.5 (Pin_5); no longer J16.1 (Pin_1)
- net A3: now also J10.6 (Pin_6); no longer J15.1 (Pin_1)
- net A4: now also J13.1 (Pin_1), J10.7 (Pin_7); no longer J4.1 (Pin_1)
- net A5: now also J14.1 (Pin_1), J10.8 (Pin_8); no longer J4.2 (Pin_2)
- net A6: now also J16.1 (Pin_1), J4.1 (Pin_1); no longer J4.3 (Pin_3)
- net A7: now also J15.1 (Pin_1), J4.2 (Pin_2); no longer J4.4 (Pin_4)
- net A8: now also J4.3 (Pin_3), J20.1 (Pin_1); no longer J4.5 (Pin_5)
- net A9: now also J4.4 (Pin_4); no longer J4.6 (Pin_6)
- net D23: now also J19.4 (Pin_4); no longer J12.1 (Pin_1)
- net D25: now also J19.3 (Pin_3); no longer J12.2 (Pin_2)
- net D27: now also J6.8 (Pin_8)
- net D29: now also J6.7 (Pin_7)
- net D31: now also J6.6 (Pin_6); no longer J6.8 (Pin_8)
- net D33: now also J6.5 (Pin_5); no longer J6.7 (Pin_7)
- net D35: now also J6.4 (Pin_4); no longer J6.6 (Pin_6)
- net D37: now also J6.3 (Pin_3); no longer J6.5 (Pin_5)
- net D39: now also J6.2 (Pin_2); no longer J6.4 (Pin_4)
- net D41: now also J6.1 (Pin_1); no longer J6.3 (Pin_3)
- net D43: now also J12.4 (Pin_4); no longer J6.2 (Pin_2)
- net D44: now also J8.1 (Pin_1)
- net D45: now also J12.3 (Pin_3); no longer J6.1 (Pin_1)
- net D46: now also J8.2 (Pin_2)
- net D50: now also J5.3 (Pin_3); no longer J5.5 (Pin_5)
- net D52: now also J5.4 (Pin_4)
- net D53: now also J5.5 (Pin_5)
- net GND: now also J12.1 (Pin_1), J18.2 (Pin_2), XA1.GND1 (GND), XA1.GND2 (GND), XA1.GND3 (GND), XA1.GND5 (GND), XA1.GND6 (GND), J10.2 (Pin_2), J19.1 (Pin_1), J20.3 (Pin_3); no longer J12.4 (Pin_4), J18.1 (Pin_1)
- net SCL: now also J11.3 (Pin_3); no longer J11.4 (Pin_4)
- net SDA: now also J11.4 (Pin_4); no longer J11.3 (Pin_3)
