File: motor driver/motor driver.sch (KiCad schematic (older format))
At the start: 49 parts, among them J1 M1, J2 M3, J3 JST IN, J5 M2, J6 M4, J7 Solar Connector, U1 L298HN, U2 L298HN, U3 L7805, U4 74HC04

Commit message: mega shield sch done
Parts:
- F1: footprint Fuse:Fuseholder_Cylinder-5x20mm_Schurter_0031_8201_Horizontal_Open -> rashik:fuse_holder
Changed lines of the file:
@@
 F 0 "F1" V 10953 2800 50  0000 C CNN
 F 1 "Fuse" V 11044 2800 50  0000 C CNN
-F 2 "Fuse:Fuseholder_Cylinder-5x20mm_Schurter_0031_8201_Horizontal_Open" V 11080 2800 50  0001 C CNN
+F 2 "rashik:fuse_holder" V 11080 2800 50  0001 C CNN
 F 3 "~" H 11150 2800 50  0001 C CNN
 	1    11150 2800

Commit message: motor driver done
Parts:
- removed C9: 220uF, Capacitor_THT:CP_Radial_D5.0mm_P2.50mm, symbol Device:CP
- removed J7: Solar Connector, rashik:Screw_Terminal_2_Pin, symbol Connector:Conn_01x02_Female
- removed U3: L7805, rashik:TO-220-3_Vertical, symbol Regulator_Linear:L7805
- added J4: Solar Conn, rashik:Screw_Terminal_3_Pin, symbol Connector:Conn_01x03_Female
- C8: value 10uF -> 100uF
Connections:
- net +12V: no longer D26.1 (K)
- net +5V: now also D26.2 (A), J4.3 (Pin_3)
- net GND: now also D26.1 (K), J4.2 (Pin_2)
- net at F1.2: now also J4.1 (Pin_1)
Other:
- moved on the sheet: C8, D26
Changed lines of the file:
@@
 Connection ~ 8800 6650
-$Comp
-L Connector:Conn_01x02_Female J7
-U 1 1 5D01191C
-P 10550 2900
-F 0 "J7" H 10442 2575 50  0000 C CNN
-F 1 "Solar Connector" H 10442 2666 50  0000 C CNN
-F 2 "rashik:Screw_Terminal_2_Pin" H 10550 2900 50  0001 C CNN
-F 3 "~" H 10550 2900 50  0001 C CNN
-	1    10550 2900
-	-1   0    0    1
-$EndComp
 $Comp
 L Device:Fuse F1
@@
 	0    1    1    0
 $EndComp
-Wire Wire Line
-	10750 2800 11000 2800
-$Comp
-L power:GND #PWR012
-U 1 1 5D030808
-P 10800 2950
-F 0 "#PWR012" H 10800 2700 50  0001 C CNN
-F 1 "GND" H 10805 2777 50  0000 C CNN
-F 2 "" H 10800 2950 50  0001 C CNN
-F 3 "" H 10800 2950 50  0001 C CNN
-	1    10800 2950
-	1    0    0    -1
-$EndComp
-Wire Wire Line
-	10750 2900 10800 2900
-Wire Wire Line
-	10800 2900 10800 2950
 $Comp
 L Device:LED D11
@@
 Connection ~ 11400 2800
 $Comp
-L Regulator_Linear:L7805 U3
-U 1 1 5D068B12
-P 11350 4150
-F 0 "U3" H 11350 4392 50  0000 C CNN
-F 1 "L7805" H 11350 4301 50  0000 C CNN
-F 2 "rashik:TO-220-3_Vertical" H 11375 4000 50  0001 L CIN
-F 3 "http://www.st.com/content/ccc/resource/technical/document/datasheet/41/4f/b3/b0/12/d4/47/88/CD00000444.pdf/files/CD00000444.pdf/jcr:content/translations/en.CD00000444.pdf" H 11350 4100 50  0001 C CNN
-	1    11350 4150
-	1    0    0    -1
-$EndComp
-$Comp
 L Device:LED D27
 U 1 1 5D06B1E9
@@
 L power:GND #PWR016
 U 1 1 5D06B1F6
-P 11350 4850
-F 0 "#PWR016" H 11350 4600 50  0001 C CNN
-F 1 "GND" H 11355 4677 50  0000 C CNN
-F 2 "" H 11350 4850 50  0001 C CNN
-F 3 "" H 11350 4850 50  0001 C CNN
-	1    11350 4850
-	1    0    0    -1
-$EndComp
-Wire Wire Line
-	11650 4150 11800 4150
+P 11700 4850
+F 0 "#PWR016" H 11700 4600 50  0001 C CNN
+F 1 "GND" H 11705 4677 50  0000 C CNN
+F 2 "" H 11700 4850 50  0001 C CNN
+F 3 "" H 11700 4850 50  0001 C CNN
+	1    11700 4850
+	1    0    0    -1
+$EndComp
 $Comp
 L power:+5V #PWR015
@@
 Connection ~ 12150 4150
 Wire Wire Line
-	11350 4450 11350 4850
-Wire Wire Line
-	11350 4850 11800 4850
-Wire Wire Line
 	12150 4850 12150 4800
-Connection ~ 11350 4850
 $Comp
 L pspice:DIODE D26
 U 1 1 5D09C645
-P 10550 4150
-F 0 "D26" H 10550 4415 50  0000 C CNN
-F 1 "DIODE" H 10550 4324 50  0000 C CNN
-F 2 "Diode_THT:D_A-405_P10.16mm_Horizontal" H 10550 4150 50  0001 C CNN
-F 3 "~" H 10550 4150 50  0001 C CNN
-	1    10550 4150
-	1    0    0    -1
-$EndComp
-Wire Wire Line
-	10750 4150 10900 4150
-$Comp
-L power:+12V #PWR014
-U 1 1 5D0A78C5
-P 10150 4150
-F 0 "#PWR014" H 10150 4000 50  0001 C CNN
-F 1 "+12V" H 10165 4323 50  0000 C CNN
-F 2 "" H 10150 4150 50  0001 C CNN
-F 3 "" H 10150 4150 50  0001 C CNN
-	1    10150 4150
-	1    0    0    -1
-$EndComp
-Wire Wire Line
-	10150 4150 10350 4150
-$Comp
-L Device:CP C9
-U 1 1 5D0B3579
-P 10900 4550
-F 0 "C9" H 11018 4596 50  0000 L CNN
-F 1 "220uF" H 11018 4505 50  0000 L CNN
-F 2 "Capacitor_THT:CP_Radial_D5.0mm_P2.50mm" H 10938 4400 50  0001 C CNN
-F 3 "~" H 10900 4550 50  0001 C CNN
-	1    10900 4550
-	1    0    0    -1
-$EndComp
-Wire Wire Line
-	10900 4150 10900 4400
-Connection ~ 10900 4150
-Wire Wire Line
-	10900 4150 11050 4150
-Wire Wire Line
-	10900 4700 10900 4850
-Wire Wire Line
-	10900 4850 11350 4850
+P 11300 4500
+F 0 "D26" H 11300 4765 50  0000 C CNN
+F 1 "DIODE" H 11300 4674 50  0000 C CNN
+F 2 "Diode_THT:D_A-405_P10.16mm_Horizontal" H 11300 4500 50  0001 C CNN
+F 3 "~" H 11300 4500 50  0001 C CNN
+	1    11300 4500
+	0    -1   -1   0
+$EndComp
 $Comp
 L Device:CP C8
 U 1 1 5D0CA06A
-P 11800 4500
-F 0 "C8" H 11918 4546 50  0000 L CNN
-F 1 "10uF" H 11918 4455 50  0000 L CNN
-F 2 "Capacitor_THT:CP_Radial_D5.0mm_P2.50mm" H 11838 4350 50  0001 C CNN
-F 3 "~" H 11800 4500 50  0001 C CNN
-	1    11800 4500
-	1    0    0    -1
-$EndComp
-Wire Wire Line
-	11800 4150 11800 4350
-Connection ~ 11800 4150
-Wire Wire Line
-	11800 4150 12150 4150
-Wire Wire Line
-	11800 4650 11800 4850
-Connection ~ 11800 4850
-Wire Wire Line
-	11800 4850 12150 4850
+P 11700 4500
+F 0 "C8" H 11818 4546 50  0000 L CNN
+F 1 "100uF" H 11818 4455 50  0000 L CNN
+F 2 "Capacitor_THT:CP_Radial_D5.0mm_P2.50mm" H 11738 4350 50  0001 C CNN
+F 3 "~" H 11700 4500 50  0001 C CNN
+	1    11700 4500
+	1    0    0    -1
+$EndComp
 $Comp
 L power:+5V #PWR017
@@
 Text Notes 10900 8900 0    157  ~ 31
 JST
+$Comp
+L power:+5V #PWR0101
+U 1 1 5CE921C0
+P 10950 2600
+F 0 "#PWR0101" H 10950 2450 50  0001 C CNN
+F 1 "+5V" H 10965 2773 50  0000 C CNN
+F 2 "" H 10950 2600 50  0001 C CNN
+F 3 "" H 10950 2600 50  0001 C CNN
+	1    10950 2600
+	1    0    0    -1
+$EndComp
+Wire Wire Line
+	11300 4300 11300 4150
+Wire Wire Line
+	11300 4700 11300 4850
+Wire Wire Line
+	11300 4850 11700 4850
+Wire Wire Line
+	11300 4150 11700 4150
+Wire Wire Line
+	11700 4350 11700 4150
+Connection ~ 11700 4150
+Wire Wire Line
+	11700 4150 12150 4150
+Wire Wire Line
+	11700 4650 11700 4850
+Connection ~ 11700 4850
+Wire Wire Line
+	11700 4850 12150 4850
+Wire Wire Line
+	10750 2600 10950 2600
+$Comp
+L Connector:Conn_01x03_Female J4
+U 1 1 5CE8EA2E
+P 10550 2700
+F 0 "J4" H 10442 2375 50  0000 C CNN
+F 1 "Solar Conn" H 10442 2466 50  0000 C CNN
+F 2 "rashik:Screw_Terminal_3_Pin" H 10550 2700 50  0001 C CNN
+F 3 "~" H 10550 2700 50  0001 C CNN
+	1    10550 2700
+	-1   0    0    1
+$EndComp
+$Comp
+L power:GND #PWR012
+U 1 1 5D030808
+P 10750 2700
+F 0 "#PWR012" H 10750 2450 50  0001 C CNN
+F 1 "GND" H 10755 2527 50  0000 C CNN
+F 2 "" H 10750 2700 50  0001 C CNN
+F 3 "" H 10750 2700 50  0001 C CNN
+	1    10750 2700
+	0    -1   -1   0
+$EndComp
+Wire Wire Line
+	10750 2800 11000 2800
 $EndSCHEMATC
